File: board/ttydriver01.kicad_pcb (KiCad board)
At the start: 2 copper layers, 119.4 x 74.9 mm, 63 parts, among them J1 PRINTER JACK, J2 KEYBOARD JACK, J3 MOTOR CTL RELAY JACK, P1 CONN_01X02, SW1 Switch_SPDT, SW2 Button_SPDT, T1 Coilcraft-FA2469-AL, U1 NE555, U2 AP2553W6, U3 CP2102-breakout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

Commit message: Successful routing - needs final check
Parts:
- removed D5: D, Diodes_SMD:SMA_Standard
- removed D8: Schottky, Diodes_SMD:SOD-323
- added C11: 1uf, Capacitors_ThroughHole:C_Disc_D6.0mm_W4.4mm_P5.00mm, F.Cu at (103.4, 131.1)
- added C13: 22uf, Capacitors_SMD:C_0805, F.Cu at (146.3, 129.0)
- added C14: 470uf, Capacitors_ThroughHole:CP_Radial_D10.0mm_P5.00mm, F.Cu at (140.7, 104.9)
- added R18: 2.2, Resistors_SMD:R_1206, F.Cu at (146.1, 121.2)
- added R2: 2.2, Resistors_SMD:R_1206, F.Cu at (146.1, 115.8)
- C9: value 220uf -> 470uf; footprint Capacitors_ThroughHole:C_Radial_D8_L11.5_P3.5 -> Capacitors_ThroughHole:CP_Radial_D10.0mm_P5.00mm
- R8: value 10K -> 2.2K
- moved R9 16.0 mm to (160.3, 120.9)
- moved U4 8.65 mm to (92.5, 137.9), turned to 0 degrees
- moved D1 4.13 mm to (114.3, 124.2)
- moved C2 1.63 mm to (112.3, 131.1)
- moved D7 1.02 mm to (119.6, 142.7)
- moved D11 0.76 mm to (89.9, 110.7), turned to 0 degrees
- moved D6 0.25 mm to (105.9, 124.2)
- turned D2 to 0 degrees
Connections:
- C2 pad 1: Net-(C2-Pad1) -> Net-(C11-Pad1)
- C9 pad 1: Net-(C1-Pad1) -> Net-(C9-Pad1)
- D1 pad 1: Net-(C2-Pad1) -> Net-(C11-Pad1)
- D2 pad 1: Net-(C1-Pad1) -> Net-(C13-Pad1)
- D6 pad 1: Net-(D5-Pad1) -> Net-(C11-Pad1)
- D7 pad 1: Net-(C2-Pad1) -> Net-(C11-Pad1)
- D9 pad 1: Net-(D8-Pad1) -> Net-(C8-Pad1)
- R12 pad 2: Net-(C1-Pad1) -> Net-(C13-Pad1)
- R14 pad 1: Net-(C2-Pad1) -> Net-(C11-Pad1)
- R6 pad 2: Net-(C1-Pad1) -> Net-(C13-Pad1)
- U1 pad 2: Net-(D8-Pad1) -> Net-(C8-Pad1)
- U1 pad 4: Net-(C1-Pad1) -> Net-(C13-Pad1)
- U1 pad 8: Net-(C1-Pad1) -> Net-(C13-Pad1)
- U2 pad 6: Net-(C1-Pad1) -> Net-(C13-Pad1)
- U3 pad 2-4: Net-(C1-Pad1) -> Net-(C13-Pad1)
- U4 pad 4: Net-(D5-Pad1) -> Net-(C11-Pad1)
- U4 pad 6: Net-(D5-Pad1) -> Net-(C11-Pad1)
- U5 pad 2: Net-(C1-Pad1) -> Net-(C13-Pad1)
- U6 pad 4: Net-(C1-Pad1) -> Net-(C13-Pad1)
- U6 pad 6: Net-(C1-Pad1) -> Net-(C13-Pad1)
- U7 pad 4: Net-(C1-Pad1) -> Net-(C13-Pad1)
- U7 pad 6: Net-(C1-Pad1) -> Net-(C13-Pad1)
- U8 pad 2: Net-(C1-Pad1) -> Net-(C13-Pad1)
- W1 pad 1: Net-(C1-Pad1) -> Net-(C13-Pad1)
- W3 pad 1: Net-(C2-Pad1) -> Net-(C11-Pad1)
Routing:
- net GND: track 395.1 -> 0.00 mm, vias 1 -> 0
- net Net-(C1-Pad1): track 254.5 -> 0.00 mm, vias 1 -> 0
- net /TxD: track 160.7 -> 0.00 mm, vias 1 -> 0
- net /HVNEG: track 152.9 -> 0.00 mm
- net Net-(J3-PadT): track 130.5 -> 0.00 mm
- net Net-(J2-PadS): track 102.5 -> 0.00 mm
- net Net-(R9-Pad1): track 99.3 -> 0.00 mm, vias 1 -> 0
- net Net-(SW1-Pad2): track 94.4 -> 0.00 mm
- net Net-(C3-Pad1): track 93.4 -> 0.00 mm
- net /ENABLE: track 78.0 -> 0.00 mm
- net /RxD: track 59.8 -> 0.00 mm
- net Net-(C10-Pad1): track 56.7 -> 0.00 mm, vias 2 -> 0
- net Net-(R13-Pad2): track 50.1 -> 0.00 mm, vias 1 -> 0
- net Net-(D9-Pad2): track 44.3 -> 0.00 mm
- net Net-(D5-Pad1): track 42.4 -> 0.00 mm
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Other:
- board text added: "Jumper OUT for 55 ohm selector"
- board text removed: "Jumper IN for 55 ohm selector"
